File: Power Testing board.kicad_sch (KiCad schematic)
At the start: 96 parts, among them J1 J_ATX_PWR: 3V3 3V3 5V 5V 12V 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, J2 J_ATX_CTRL: PS_ON PWR_OK 5VSB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, J3 ATX_SWITCH, J4 DEDICATED OUTPUTS: 3V3/G 5V/G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, Q1 2N7002 RESET_3V3 pulldown, Q2 2N7002 RESET_5V pulldown, Q3 2N7002 RESET_12V pulldown, Q4 2N7002 RESET_16V8 pulldown, Q5 2N7002 ATX PS_ON# pulldown, SW1 RESET_3V3 edge button, SW2 RESET_5V edge button, SW3 RESET_12V edge button, SW4 RESET_16V8 edge button, U1 TPS259814L 3V3 eFuse latch-off, U2 TPS26631RGE 5V eFuse, U3 TPS26631RGE 12V eFuse, U4 TPS26631RGE 16V8 eFuse, U5 INA260 3V3 module, U6 INA260 5V module, U7 INA260 12V module, U8 INA260 16V8 module, U9 Boost 12V to 16.8V module 60x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

Commit message: chat
Other:
- note added: "+12V_PROTECTED branches only after INA260 VIN-"
- note added: "+16V8_PROTECTED branches only after INA260 VIN-"
- note added: "+3V3_PROTECTED branches only after INA260 VIN-"
- note added: "+5V_PROTECTED branches only after INA260 VIN-"
- note added: "12V rail: RAW/source -> eFuse -> INA260 VIN+ / VIN- -> protected bus"
- note added: "16.8V rail: RAW/source -> eFuse -> INA260 VIN+ / VIN- -> protected bus"
- note added: "3.3V rail: RAW/source -> eFuse -> INA260 VIN+ / VIN- -> protected bus"
- note added: "4-layer PCB intent: L1 components/high-current/local signals, L2 solid GND reference, L3 power zones, L4 secondary routing/GND fill."
- note added: "5V rail: RAW/source -> eFuse -> INA260 VIN+ / VIN- -> protected bus"
- note added: "ATX input and control terminals"
- note added: "Arduino/control section: USB-powered Nano, open-drain reset MOSFETs, FLT inputs, PS_ON# pulldown"
- note added: "Boost module: verified 60 mm x 42 mm x 20 mm footprint, +12V in and +16.8V out"
- note added: "Edge-access reset buttons: RESET_3V3, RESET_5V, RESET_12V, RESET_16V8"
- note added: "Only user-selected H1/H2 mission power and GND pins are connected. Excluded communication/normally-closed pins are not represented here."
- note added: "Output connectors: dedicated terminal J4 plus selected EPS H1/H2 power/GND pins only"
- note added: "Protected rail chains"
- note added: "Serviceable layout choice: eFuse ICs are on the main PCB for manufacturer assembly. For true field replacement, move each eFuse circuit to a plug-in daughterboard."
- note added: "Test points"
- note removed: "Boost module footprint uses physically verified 60 mm x 42 mm x 20 mm module geometry."
- note removed: "Only user-selected H1/H2 mission power and GND pins are connected. Excluded/communication pins are not represented in this schematic."
- note removed: "Serviceable layout choice: eFuse ICs are on the main PCB for manufacturer assembly. If field replacement becomes more important than board area, move each eFuse circuit to a plug-in daughterboard."
- title: Compact CubeSat EPS Power Testing Board -> CubeSat EPS Power Testing Board - 4 Layer Revision

Commit message: test
Parts:
- removed A1: Arduino Nano USB-powered socket, Module:Arduino_Nano, symbol Power_Testing_Board:Arduino_Nano_USB_Powered
- removed C1, C3: 1uF 25V X7R input close to eFuse, Capacitor_SMD:C_0805_2012Metric, symbol Power_Testing_Board:C
- removed C2, C4: 10uF 25V X7R output close to eFuse, Capacitor_SMD:C_0805_2012Metric, symbol Power_Testing_Board:C
- removed C5, C7: 1uF 50V X7R input close to eFuse, Capacitor_SMD:C_0805_2012Metric, symbol Power_Testing_Board:C
- removed C6, C8: 10uF 50V X7R output close to eFuse, Capacitor_SMD:C_0805_2012Metric, symbol Power_Testing_Board:C
- removed J1: J_ATX_PWR: 3V3 3V3 5V 5V 12V 12V GNDx4, TerminalBlock:TerminalBlock_MaiXu_MX126-5.0-10P_1x10_P5.00mm, symbol Power_Testing_Board:Conn_01x10
- removed J2: J_ATX_CTRL: PS_ON PWR_OK 5VSB GND, TerminalBlock:TerminalBlock_MaiXu_MX126-5.0-04P_1x04_P5.00mm, symbol Power_Testing_Board:Conn_01x04
- removed J3: ATX_SWITCH, TerminalBlock:TerminalBlock_MaiXu_MX126-5.0-02P_1x02_P5.00mm, symbol Power_Testing_Board:Conn_01x02
- removed J4: DEDICATED OUTPUTS: 3V3/G 5V/G 12V/G 16V8/G, TerminalBlock:TerminalBlock_MaiXu_MX126-5.0-08P_1x08_P5.00mm, symbol Power_Testing_Board:Conn_01x08
- removed JH1: H1 selected power/GND pins only, Connector_PinSocket_2.54mm:PinSocket_2x26_P2.54mm_Vertical, symbol Power_Testing_Board:PC104_H1_SelectedPowerPins
- removed JH2: H2 selected power/GND pins only, Connector_PinSocket_2.54mm:PinSocket_2x26_P2.54mm_Vertical, symbol Power_Testing_Board:PC104_H2_SelectedPowerPins
- removed Q1: 2N7002 RESET_3V3 pulldown, Package_TO_SOT_SMD:SOT-23, symbol Power_Testing_Board:NMOS_GSD
- removed Q2: 2N7002 RESET_5V pulldown, Package_TO_SOT_SMD:SOT-23, symbol Power_Testing_Board:NMOS_GSD
- removed Q3: 2N7002 RESET_12V pulldown, Package_TO_SOT_SMD:SOT-23, symbol Power_Testing_Board:NMOS_GSD
- removed Q4: 2N7002 RESET_16V8 pulldown, Package_TO_SOT_SMD:SOT-23, symbol Power_Testing_Board:NMOS_GSD
- removed Q5: 2N7002 ATX PS_ON# pulldown, Package_TO_SOT_SMD:SOT-23, symbol Power_Testing_Board:NMOS_GSD
- removed R1: 1.10k 1% ILM ~6A, Resistor_SMD:R_0805_2012Metric, symbol Power_Testing_Board:R
- removed R10: 261k 1% UVLO top 4.33V, Resistor_SMD:R_0603_1608Metric, symbol Power_Testing_Board:R
- removed R11, R19, R27: 100k 1% UVLO bottom, Resistor_SMD:R_0603_1608Metric, symbol Power_Testing_Board:R
- removed R12: 383k 1% OVP top 5.80V, Resistor_SMD:R_0603_1608Metric, symbol Power_Testing_Board:R
- removed R13, R21, R29: 100k 1% OVP bottom, Resistor_SMD:R_0603_1608Metric, symbol Power_Testing_Board:R
- removed R14, R22, R30, R33, R6: 330 gate, Resistor_SMD:R_0603_1608Metric, symbol Power_Testing_Board:R
- removed R15, R23, R31, R34, R7: 100k gate pulldown, Resistor_SMD:R_0603_1608Metric, symbol Power_Testing_Board:R
- removed R16, R24, R32, R8: 10k FLT pullup, Resistor_SMD:R_0603_1608Metric, symbol Power_Testing_Board:R
- removed R17, R25, R9: 3.00k 1% ILIM ~6A, Resistor_SMD:R_0805_2012Metric, symbol Power_Testing_Board:R
- removed R18: 806k 1% UVLO top 10.87V, Resistor_SMD:R_0603_1608Metric, symbol Power_Testing_Board:R
- removed R2: 100k 1% EN top 2.40V, Resistor_SMD:R_0603_1608Metric, symbol Power_Testing_Board:R
- removed R20: 1.05M 1% OVP top 13.80V, Resistor_SMD:R_0603_1608Metric, symbol Power_Testing_Board:R
- removed R26: 1.07M 1% UVLO top 14.04V, Resistor_SMD:R_0603_1608Metric, symbol Power_Testing_Board:R
- removed R28: 1.40M 1% OVP top 18.00V, Resistor_SMD:R_0603_1608Metric, symbol Power_Testing_Board:R
- removed R3: 100k 1% EN bottom, Resistor_SMD:R_0603_1608Metric, symbol Power_Testing_Board:R
- removed R4: 24.9k 1% OVLO top 4.19V, Resistor_SMD:R_0603_1608Metric, symbol Power_Testing_Board:R
- removed R5: 10k 1% OVLO bottom, Resistor_SMD:R_0603_1608Metric, symbol Power_Testing_Board:R
- removed SW1: RESET_3V3 edge button, Button_Switch_THT:SW_PUSH_6mm, symbol Power_Testing_Board:SW_Push
- removed SW2: RESET_5V edge button, Button_Switch_THT:SW_PUSH_6mm, symbol Power_Testing_Board:SW_Push
- removed SW3: RESET_12V edge button, Button_Switch_THT:SW_PUSH_6mm, symbol Power_Testing_Board:SW_Push
- removed SW4: RESET_16V8 edge button, Button_Switch_THT:SW_PUSH_6mm, symbol Power_Testing_Board:SW_Push
- removed TP1: +3V3_RAW, TestPoint:TestPoint_Pad_D1.0mm, symbol Power_Testing_Board:TP
- removed TP10: +16V8_RAW, TestPoint:TestPoint_Pad_D1.0mm, symbol Power_Testing_Board:TP
- removed TP11: +16V8_EFUSE_OUT, TestPoint:TestPoint_Pad_D1.0mm, symbol Power_Testing_Board:TP
- removed TP12: +16V8_PROTECTED, TestPoint:TestPoint_Pad_D1.0mm, symbol Power_Testing_Board:TP
- removed TP13: GND, TestPoint:TestPoint_Pad_D1.0mm, symbol Power_Testing_Board:TP
- removed TP14: I2C_SDA, TestPoint:TestPoint_Pad_D1.0mm, symbol Power_Testing_Board:TP
- removed TP15: I2C_SCL, TestPoint:TestPoint_Pad_D1.0mm, symbol Power_Testing_Board:TP
- removed TP16: ATX_PS_ON_N, TestPoint:TestPoint_Pad_D1.0mm, symbol Power_Testing_Board:TP
- removed TP17: ATX_PWR_OK, TestPoint:TestPoint_Pad_D1.0mm, symbol Power_Testing_Board:TP
- removed TP18: +5VSB, TestPoint:TestPoint_Pad_D1.0mm, symbol Power_Testing_Board:TP
- removed TP19: RESET_3V3, TestPoint:TestPoint_Pad_D1.0mm, symbol Power_Testing_Board:TP
- removed TP2: +3V3_EFUSE_OUT, TestPoint:TestPoint_Pad_D1.0mm, symbol Power_Testing_Board:TP
- removed TP20: RESET_5V, TestPoint:TestPoint_Pad_D1.0mm, symbol Power_Testing_Board:TP
- removed TP21: RESET_12V, TestPoint:TestPoint_Pad_D1.0mm, symbol Power_Testing_Board:TP
- removed TP22: RESET_16V8, TestPoint:TestPoint_Pad_D1.0mm, symbol Power_Testing_Board:TP
- removed TP23: FLT_3V3, TestPoint:TestPoint_Pad_D1.0mm, symbol Power_Testing_Board:TP
- removed TP24: FLT_5V, TestPoint:TestPoint_Pad_D1.0mm, symbol Power_Testing_Board:TP
- removed TP25: FLT_12V, TestPoint:TestPoint_Pad_D1.0mm, symbol Power_Testing_Board:TP
- removed TP26: FLT_16V8, TestPoint:TestPoint_Pad_D1.0mm, symbol Power_Testing_Board:TP
- removed TP27: BOOST_IN+ (+12V_RAW), TestPoint:TestPoint_Pad_D1.0mm, symbol Power_Testing_Board:TP
- removed TP28: BOOST_OUT+ (+16V8_RAW), TestPoint:TestPoint_Pad_D1.0mm, symbol Power_Testing_Board:TP
- removed TP29: BOOST_GND, TestPoint:TestPoint_Pad_D1.0mm, symbol Power_Testing_Board:TP
- removed TP3: +3V3_PROTECTED, TestPoint:TestPoint_Pad_D1.0mm, symbol Power_Testing_Board:TP
- removed TP4: +5V_RAW, TestPoint:TestPoint_Pad_D1.0mm, symbol Power_Testing_Board:TP
- removed TP5: +5V_EFUSE_OUT, TestPoint:TestPoint_Pad_D1.0mm, symbol Power_Testing_Board:TP
- removed TP6: +5V_PROTECTED, TestPoint:TestPoint_Pad_D1.0mm, symbol Power_Testing_Board:TP
- removed TP7: +12V_RAW, TestPoint:TestPoint_Pad_D1.0mm, symbol Power_Testing_Board:TP
- removed TP8: +12V_EFUSE_OUT, TestPoint:TestPoint_Pad_D1.0mm, symbol Power_Testing_Board:TP
- removed TP9: +12V_PROTECTED, TestPoint:TestPoint_Pad_D1.0mm, symbol Power_Testing_Board:TP
- removed U1: TPS259814L 3V3 eFuse latch-off, Package_DFN_QFN:Texas_RPU0010A_VQFN-HR-10_2x2mm_P0.5mm, symbol Power_Testing_Board:TPS259814L_RPW_eFuse
- removed U2: TPS26631RGE 5V eFuse, Package_DFN_QFN:Texas_RGE0024H_VQFN-24-1EP_4x4mm_P0.5mm_EP2.7x2.7mm_ThermalVias, symbol Power_Testing_Board:TPS26631RGE_eFuse
- removed U3: TPS26631RGE 12V eFuse, Package_DFN_QFN:Texas_RGE0024H_VQFN-24-1EP_4x4mm_P0.5mm_EP2.7x2.7mm_ThermalVias, symbol Power_Testing_Board:TPS26631RGE_eFuse
- removed U4: TPS26631RGE 16V8 eFuse, Package_DFN_QFN:Texas_RGE0024H_VQFN-24-1EP_4x4mm_P0.5mm_EP2.7x2.7mm_ThermalVias, symbol Power_Testing_Board:TPS26631RGE_eFuse
- removed U5: INA260 3V3 module, Power_Testing_Board:Adafruit_INA260_4226_Module, symbol Power_Testing_Board:Adafruit_INA260_4226_Module
- removed U6: INA260 5V module, Power_Testing_Board:Adafruit_INA260_4226_Module, symbol Power_Testing_Board:Adafruit_INA260_4226_Module
- removed U7: INA260 12V module, Power_Testing_Board:Adafruit_INA260_4226_Module, symbol Power_Testing_Board:Adafruit_INA260_4226_Module
- removed U8: INA260 16V8 module, Power_Testing_Board:Adafruit_INA260_4226_Module, symbol Power_Testing_Board:Adafruit_INA260_4226_Module
- removed U9: Boost 12V to 16.8V module 60x42 VERIFIED, Power_Testing_Board:Boost_Module_60x42_VERIFIED, symbol Power_Testing_Board:Boost_Module_60x42
Connections:
- no-connect marks 25 -> 0
Other:
- added sheet PTB1 Schematic 1 (PTB1Schem1.kicad_sch)
- added sheet PTB1 Schematic 2 (PTB1Schem2.kicad_sch)
- note removed: "+12V_PROTECTED branches only after INA260 VIN-"
- note removed: "+16V8_PROTECTED branches only after INA260 VIN-"
- note removed: "+3V3_PROTECTED branches only after INA260 VIN-"
- note removed: "+5V_PROTECTED branches only after INA260 VIN-"
- note removed: "12V rail: RAW/source -> eFuse -> INA260 VIN+ / VIN- -> protected bus"
- note removed: "16.8V rail: RAW/source -> eFuse -> INA260 VIN+ / VIN- -> protected bus"
- note removed: "3.3V rail: RAW/source -> eFuse -> INA260 VIN+ / VIN- -> protected bus"
- note removed: "4-layer PCB intent: L1 components/high-current/local signals, L2 solid GND reference, L3 power zones, L4 secondary routing/GND fill."
- note removed: "5V rail: RAW/source -> eFuse -> INA260 VIN+ / VIN- -> protected bus"
- note removed: "ATX input and control terminals"
- note removed: "Arduino/control section: USB-powered Nano, open-drain reset MOSFETs, FLT inputs, PS_ON# pulldown"
- note removed: "Boost module: verified 60 mm x 42 mm x 20 mm footprint, +12V in and +16.8V out"
- note removed: "Edge-access reset buttons: RESET_3V3, RESET_5V, RESET_12V, RESET_16V8"
- note removed: "Only user-selected H1/H2 mission power and GND pins are connected. Excluded communication/normally-closed pins are not represented here."
- note removed: "Output connectors: dedicated terminal J4 plus selected EPS H1/H2 power/GND pins only"
- note removed: "Power path on every rail: RAW -> eFuse -> INA260 VIN+ -> INA260 VIN- -> PROTECTED output. INA260 VIN- is the downstream positive rail, never GND."
- note removed: "Protected rail chains"
- note removed: "Serviceable layout choice: eFuse ICs are on the main PCB for manufacturer assembly. For true field replacement, move each eFuse circuit to a plug-in daughterboard."
- note removed: "Test points"
- company: CSULB SHARKSAT TEAM -> (none)
- title: CubeSat EPS Power Testing Board - 4 Layer Revision -> Power Testing Board
