File: Headers.kicad_sch (KiCad schematic)
At the start: 0 parts

Commit message: page
Parts:
- added J1, J2, J3, J4: Conn_01x26_Pin, Connector_PinHeader_2.54mm:PinHeader_1x26_P2.54mm_Vertical, symbol Connector:Conn_01x26_Pin
