File: Power Testing board.kicad_pcb (KiCad board)
At the start: 2 copper layers, 230 x 170 mm, 96 parts, among them J1 J_ATX_PWR: 3V3 3V3 5V 5V 12V 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, J2 J_ATX_CTRL: PS_ON PWR_OK 5VSB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, J3 ATX_SWITCH, J4 DEDICATED OUTPUTS: 3V3/G 5V/G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, Q1 2N7002 RESET_3V3 pulldown, Q2 2N7002 RESET_5V pulldown, Q3 2N7002 RESET_12V pulldown, Q4 2N7002 RESET_16V8 pulldown, Q5 2N7002 ATX PS_ON# pulldown, SW1 RESET_3V3 edge button, SW2 RESET_5V edge button, SW3 RESET_12V edge button, SW4 RESET_16V8 edge button, U1 TPS259814L 3V3 eFuse latch-off, U2 TPS26631RGE 5V eFuse, U3 TPS26631RGE 12V eFuse, U4 TPS26631RGE 16V8 eFuse, U5 INA260 3V3 module, U6 INA260 5V module, U7 INA260 12V module, U8 INA260 16V8 module, U9 Boost 12V to 16.8V module 60x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

Commit message: chat
Parts:
- moved A1 20.0 mm to (36.0, 44.0), turned to 180 degrees
Routing:
- net UVLO_16V8: track 30.8 -> 67.1 mm
- net I2C_SDA: track 163.9 -> 196.1 mm
- net I2C_SCL: track 174.1 -> 203.8 mm
- net ATX_PWR_OK: track 177.2 -> 205.2 mm, vias 1 -> 0
- net +ARDUINO_5V: track 289.7 -> 316.0 mm
- net GND: track 1112.5 -> 1088.1 mm, vias 1 -> 3
- net ARD_RESET_3V3: track 161.8 -> 140.5 mm
- net ATX_PS_ON_CTL: track 128.2 -> 148.2 mm
- net ARD_RESET_12V: track 200.8 -> 183.3 mm
- net RESET_12V: track 116.7 -> 134.1 mm, vias 2 -> 1
- net FLT_16V8: track 172.5 -> 187.5 mm
- net FLT_3V3: track 98.5 -> 113.3 mm, vias 1 -> 2
- net ARD_RESET_5V: track 179.2 -> 164.6 mm
- net +3V3_PROTECTED: track 136.6 -> 150.3 mm
- net ARD_RESET_16V8: track 218.3 -> 206.8 mm
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- added copper zone on In2.Cu, net +12V_PROTECTED
- added copper zone on In2.Cu, net +12V_RAW
- added copper zone on In2.Cu, net +3V3_PROTECTED
- added copper zone on In2.Cu, net +3V3_RAW
- added copper zone on In2.Cu, net +5V_RAW
- added copper zone on In1.Cu, net GND
Other:
- copper layers 2 -> 4
- board text added: "ARDUINO USB EDGE"
- board text added: "EPS POWER TEST - 4 LAYER, 2 OZ OUTER Cu RECOMMENDED"
- board text removed: "EPS POWER TEST - 2 OZ Cu RECOMMENDED"

Commit message: test
Parts:
- removed A1: Arduino Nano USB-powered socket, Arduino_Nano
- removed C1, C3: 1uF 25V X7R input close to eFuse, C_0805_2012Metric
- removed C2, C4: 10uF 25V X7R output close to eFuse, C_0805_2012Metric
- removed C5, C7: 1uF 50V X7R input close to eFuse, C_0805_2012Metric
- removed C6, C8: 10uF 50V X7R output close to eFuse, C_0805_2012Metric
- removed J1: J_ATX_PWR: 3V3 3V3 5V 5V 12V 12V GNDx4, TerminalBlock_MaiXu_MX126-5.0-10P_1x10_P5.00mm
- removed J2: J_ATX_CTRL: PS_ON PWR_OK 5VSB GND, TerminalBlock_MaiXu_MX126-5.0-04P_1x04_P5.00mm
- removed J3: ATX_SWITCH, TerminalBlock_MaiXu_MX126-5.0-02P_1x02_P5.00mm
- removed J4: DEDICATED OUTPUTS: 3V3/G 5V/G 12V/G 16V8/G, TerminalBlock_MaiXu_MX126-5.0-08P_1x08_P5.00mm
- removed JH1: H1 selected power/GND pins only, PinSocket_2x26_P2.54mm_Vertical
- removed JH2: H2 selected power/GND pins only, PinSocket_2x26_P2.54mm_Vertical
- removed Q1: 2N7002 RESET_3V3 pulldown, SOT-23
- removed Q2: 2N7002 RESET_5V pulldown, SOT-23
- removed Q3: 2N7002 RESET_12V pulldown, SOT-23
- removed Q4: 2N7002 RESET_16V8 pulldown, SOT-23
- removed Q5: 2N7002 ATX PS_ON# pulldown, SOT-23
- removed R1: 1.10k 1% ILM ~6A, R_0805_2012Metric
- removed R10: 261k 1% UVLO top 4.33V, R_0603_1608Metric
- removed R11, R19, R27: 100k 1% UVLO bottom, R_0603_1608Metric
- removed R12: 383k 1% OVP top 5.80V, R_0603_1608Metric
- removed R13, R21, R29: 100k 1% OVP bottom, R_0603_1608Metric
- removed R14, R22, R30, R33, R6: 330 gate, R_0603_1608Metric
- removed R15, R23, R31, R34, R7: 100k gate pulldown, R_0603_1608Metric
- removed R16, R24, R32, R8: 10k FLT pullup, R_0603_1608Metric
- removed R17, R25, R9: 3.00k 1% ILIM ~6A, R_0805_2012Metric
- removed R18: 806k 1% UVLO top 10.87V, R_0603_1608Metric
- removed R2: 100k 1% EN top 2.40V, R_0603_1608Metric
- removed R20: 1.05M 1% OVP top 13.80V, R_0603_1608Metric
- removed R26: 1.07M 1% UVLO top 14.04V, R_0603_1608Metric
- removed R28: 1.40M 1% OVP top 18.00V, R_0603_1608Metric
- removed R3: 100k 1% EN bottom, R_0603_1608Metric
- removed R4: 24.9k 1% OVLO top 4.19V, R_0603_1608Metric
- removed R5: 10k 1% OVLO bottom, R_0603_1608Metric
- removed SW1: RESET_3V3 edge button, SW_PUSH_6mm
- removed SW2: RESET_5V edge button, SW_PUSH_6mm
- removed SW3: RESET_12V edge button, SW_PUSH_6mm
- removed SW4: RESET_16V8 edge button, SW_PUSH_6mm
- removed TP1: +3V3_RAW, TestPoint_Pad_D1.0mm
- removed TP10: +16V8_RAW, TestPoint_Pad_D1.0mm
- removed TP11: +16V8_EFUSE_OUT, TestPoint_Pad_D1.0mm
- removed TP12: +16V8_PROTECTED, TestPoint_Pad_D1.0mm
- removed TP13: GND, TestPoint_Pad_D1.0mm
- removed TP14: I2C_SDA, TestPoint_Pad_D1.0mm
- removed TP15: I2C_SCL, TestPoint_Pad_D1.0mm
- removed TP16: ATX_PS_ON_N, TestPoint_Pad_D1.0mm
- removed TP17: ATX_PWR_OK, TestPoint_Pad_D1.0mm
- removed TP18: +5VSB, TestPoint_Pad_D1.0mm
- removed TP19: RESET_3V3, TestPoint_Pad_D1.0mm
- removed TP2: +3V3_EFUSE_OUT, TestPoint_Pad_D1.0mm
- removed TP20: RESET_5V, TestPoint_Pad_D1.0mm
- removed TP21: RESET_12V, TestPoint_Pad_D1.0mm
- removed TP22: RESET_16V8, TestPoint_Pad_D1.0mm
- removed TP23: FLT_3V3, TestPoint_Pad_D1.0mm
- removed TP24: FLT_5V, TestPoint_Pad_D1.0mm
- removed TP25: FLT_12V, TestPoint_Pad_D1.0mm
- removed TP26: FLT_16V8, TestPoint_Pad_D1.0mm
- removed TP27: BOOST_IN+ (+12V_RAW), TestPoint_Pad_D1.0mm
- removed TP28: BOOST_OUT+ (+16V8_RAW), TestPoint_Pad_D1.0mm
- removed TP29: BOOST_GND, TestPoint_Pad_D1.0mm
- removed TP3: +3V3_PROTECTED, TestPoint_Pad_D1.0mm
- removed TP4: +5V_RAW, TestPoint_Pad_D1.0mm
- removed TP5: +5V_EFUSE_OUT, TestPoint_Pad_D1.0mm
- removed TP6: +5V_PROTECTED, TestPoint_Pad_D1.0mm
- removed TP7: +12V_RAW, TestPoint_Pad_D1.0mm
- removed TP8: +12V_EFUSE_OUT, TestPoint_Pad_D1.0mm
- removed TP9: +12V_PROTECTED, TestPoint_Pad_D1.0mm
- removed U1: TPS259814L 3V3 eFuse latch-off, Texas_RPU0010A_VQFN-HR-10_2x2mm_P0.5mm
- removed U2: TPS26631RGE 5V eFuse, Texas_RGE0024H_VQFN-24-1EP_4x4mm_P0.5mm_EP2.7x2.7mm_ThermalVias
- removed U3: TPS26631RGE 12V eFuse, Texas_RGE0024H_VQFN-24-1EP_4x4mm_P0.5mm_EP2.7x2.7mm_ThermalVias
- removed U4: TPS26631RGE 16V8 eFuse, Texas_RGE0024H_VQFN-24-1EP_4x4mm_P0.5mm_EP2.7x2.7mm_ThermalVias
- removed U5: INA260 3V3 module, Adafruit_INA260_4226_Module
- removed U6: INA260 5V module, Adafruit_INA260_4226_Module
- removed U7: INA260 12V module, Adafruit_INA260_4226_Module
- removed U8: INA260 16V8 module, Adafruit_INA260_4226_Module
- removed U9: Boost 12V to 16.8V module 60x42 VERIFIED, Boost_Module_60x42_VERIFIED
Routing:
- net GND: track 1088.1 -> 0.00 mm, vias 3 -> 0
- net +ARDUINO_5V: track 316.0 -> 0.00 mm
- net +12V_RAW: track 258.0 -> 0.00 mm
- net +16V8_RAW: track 212.7 -> 0.00 mm
- net ARD_RESET_16V8: track 206.8 -> 0.00 mm, vias 1 -> 0
- net ATX_PWR_OK: track 205.2 -> 0.00 mm
- net I2C_SCL: track 203.8 -> 0.00 mm
- net I2C_SDA: track 196.1 -> 0.00 mm
- net FLT_16V8: track 187.5 -> 0.00 mm, vias 1 -> 0
- net RESET_3V3: track 187.2 -> 0.00 mm, vias 2 -> 0
- net ARD_RESET_12V: track 183.3 -> 0.00 mm, vias 1 -> 0
- net +16V8_PROTECTED: track 182.3 -> 0.00 mm
- net ARD_RESET_5V: track 164.6 -> 0.00 mm, vias 1 -> 0
- net FLT_12V: track 156.1 -> 0.00 mm, vias 1 -> 0
- net +3V3_PROTECTED: track 150.3 -> 0.00 mm
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- removed copper zone on B.Cu, net +12V_EFUSE_OUT
- removed copper zone on F.Cu, net +12V_PROTECTED
- removed copper zone on In2.Cu, net +12V_PROTECTED
- removed copper zone on F.Cu, net +12V_RAW
- removed copper zone on In2.Cu, net +12V_RAW
- removed copper zone on F.Cu, net +16V8_EFUSE_OUT
- removed copper zone on B.Cu, net +16V8_PROTECTED
- removed copper zone on B.Cu, net +16V8_RAW
- removed copper zone on F.Cu, net +3V3_EFUSE_OUT
- removed copper zone on F.Cu, net +3V3_PROTECTED
- removed copper zone on In2.Cu, net +3V3_PROTECTED
- removed copper zone on F.Cu, net +3V3_RAW
- removed copper zone on In2.Cu, net +3V3_RAW
- removed copper zone on F.Cu, net +5V_EFUSE_OUT
- removed copper zone on B.Cu, net +5V_PROTECTED
- removed copper zone on B.Cu, net +5V_RAW
- removed copper zone on In2.Cu, net +5V_RAW
- removed copper zone on B.Cu, net GND
- removed copper zone on In1.Cu, net GND
Other:
- board outline removed
- copper layers 4 -> 2
- board text removed: "ARDUINO USB EDGE"
- board text removed: "ATX INPUTS"
- board text removed: "BOOST 60x42 VERIFIED"
- board text removed: "EPS POWER TEST - 4 LAYER, 2 OZ OUTER Cu RECOMMENDED"
- board text removed: "H1/H2 POWER/GND ONLY"
- board text removed: "RAW -> EFUSE -> INA260 -> OUTPUT"
- board text removed: "RESET_3V3 RESET_5V RESET_12V RESET_16V8"
