File: Power Testing board/Power Testing board.kicad_sch (KiCad schematic)
At the start: 9 parts, among them J1 Conn_01x26_Pin, J2 Conn_01x26_Pin, J3 Conn_01x26_Pin, J4 Conn_01x26_Pin, U1 INA260, U2 INA260, U3 INA260, U4 INA260

Commit message: buckboostconv
Other:
- added sheet buck_boost_converter (untitled.kicad_sch)
